File: inductor_test.sch (KiCad schematic (older format))
At the start: 37 parts, among them CON1 AVR-ISP-10, J1 DC_JACK, P1 CONN_4, P2 CONN_2, P3 CONN_2, Q1 2N7000, Q2 2N7000, Q3 2N2906, Q4 2N2222A, Q5 IRLIZ24N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

Commit message: ...
Parts:
- added C?: .47uF, symbol C
- added C?: 47pF, symbol C
Connections:
- net GND: now also C?.2, C?.2
- net Vin: now also C?.1, C?.1
Other:
- moved on the sheet: P2, P3
Changed lines of the file:
@@
 L CONN_2 P2
 U 1 1 595F3354
-P 9300 3850
-F 0 "P2" V 9250 3850 40  0000 C CNN
-F 1 "CONN_2" V 9350 3850 40  0000 C CNN
-F 2 "" H 9300 3850 60  0001 C CNN
-F 3 "" H 9300 3850 60  0001 C CNN
-	1    9300 3850
+P 9850 3850
+F 0 "P2" V 9800 3850 40  0000 C CNN
+F 1 "CONN_2" V 9900 3850 40  0000 C CNN
+F 2 "" H 9850 3850 60  0001 C CNN
+F 3 "" H 9850 3850 60  0001 C CNN
+	1    9850 3850
 	1    0    0    -1
 $EndComp
@@
 	8150 1000 8150 3800
 Wire Wire Line
-	8950 3950 8800 3950
-Wire Wire Line
-	8800 3950 8800 4150
-Wire Wire Line
-	8800 4150 8150 4150
+	9500 3950 9350 3950
+Wire Wire Line
+	9350 3950 9350 4150
+Wire Wire Line
+	9350 4150 8150 4150
 Connection ~ 8150 4150
 Connection ~ 8400 3750
@@
 L CONN_2 P3
 U 1 1 5964B59F
-P 9350 4900
-F 0 "P3" V 9300 4900 40  0000 C CNN
-F 1 "CONN_2" V 9400 4900 40  0000 C CNN
-F 2 "" H 9350 4900 60  0001 C CNN
-F 3 "" H 9350 4900 60  0001 C CNN
-	1    9350 4900
+P 9900 4900
+F 0 "P3" V 9850 4900 40  0000 C CNN
+F 1 "CONN_2" V 9950 4900 40  0000 C CNN
+F 2 "" H 9900 4900 60  0001 C CNN
+F 3 "" H 9900 4900 60  0001 C CNN
+	1    9900 4900
 	1    0    0    -1
 $EndComp
@@
 L GND #PWR017
 U 1 1 5964B6DA
+P 9550 5100
+F 0 "#PWR017" H 9550 5100 30  0001 C CNN
+F 1 "GND" H 9550 5030 30  0001 C CNN
+F 2 "" H 9550 5100 60  0000 C CNN
+F 3 "" H 9550 5100 60  0000 C CNN
+	1    9550 5100
+	1    0    0    -1
+$EndComp
+Wire Wire Line
+	9550 5000 9550 5100
+Wire Wire Line
+	8150 4700 9450 4700
+Wire Wire Line
+	9450 4700 9450 4800
+Wire Wire Line
+	9450 4800 9550 4800
+Connection ~ 8150 4700
+Wire Wire Line
+	6600 4050 7650 4050
+Wire Wire Line
+	8150 3750 9500 3750
+Wire Wire Line
+	1350 1000 8150 1000
+Wire Wire Line
+	3700 1400 3600 1400
+Wire Wire Line
+	4500 1400 7650 1400
+Wire Wire Line
+	7650 1400 7650 4050
+Connection ~ 3600 1000
+$Comp
+L C C?
+U 1 1 5964E1CA
+P 8750 4400
+F 0 "C?" H 8775 4500 50  0000 L CNN
+F 1 ".47uF" H 8775 4300 50  0000 L CNN
+F 2 "" H 8788 4250 50  0001 C CNN
+F 3 "" H 8750 4400 50  0001 C CNN
+	1    8750 4400
+	1    0    0    -1
+$EndComp
+$Comp
+L C C?
+U 1 1 5964E257
+P 9000 4400
+F 0 "C?" H 9025 4500 50  0000 L CNN
+F 1 "47pF" H 9025 4300 50  0000 L CNN
+F 2 "" H 9038 4250 50  0001 C CNN
+F 3 "" H 9000 4400 50  0001 C CNN
+	1    9000 4400
+	1    0    0    -1
+$EndComp
+Wire Wire Line
+	8750 4250 8750 3750
+Connection ~ 8750 3750
+Wire Wire Line
+	9000 3750 9000 4250
+Connection ~ 9000 3750
+$Comp
+L GND #PWR?
+U 1 1 5964E57B
+P 8750 5100
+F 0 "#PWR?" H 8750 5100 30  0001 C CNN
+F 1 "GND" H 8750 5030 30  0001 C CNN
+F 2 "" H 8750 5100 60  0000 C CNN
+F 3 "" H 8750 5100 60  0000 C CNN
+	1    8750 5100
+	1    0    0    -1
+$EndComp
+$Comp
+L GND #PWR?
+U 1 1 5964E5E1
 P 9000 5100
-F 0 "#PWR017" H 9000 5100 30  0001 C CNN
+F 0 "#PWR?" H 9000 5100 30  0001 C CNN
 F 1 "GND" H 9000 5030 30  0001 C CNN
 F 2 "" H 9000 5100 60  0000 C CNN
@@
 $EndComp
 Wire Wire Line
-	9000 5000 9000 5100
-Wire Wire Line
-	8150 4700 8900 4700
-Wire Wire Line
-	8900 4700 8900 4800
-Wire Wire Line
-	8900 4800 9000 4800
-Connection ~ 8150 4700
-Wire Wire Line
-	6600 4050 7650 4050
-Wire Wire Line
-	8150 3750 8950 3750
-Wire Wire Line
-	1350 1000 8150 1000
-Wire Wire Line
-	3700 1400 3600 1400
-Wire Wire Line
-	4500 1400 7650 1400
-Wire Wire Line
-	7650 1400 7650 4050
-Connection ~ 3600 1000
+	8750 4550 8750 5100
+Wire Wire Line
+	9000 4550 9000 5100
 $EndSCHEMATC

Commit message: ...
Parts:
- removed P3: CONN_2, symbol CONN_2
- added C2: C, symbol C
- added P3: CONN_4, Pin_Headers:Pin_Header_Angled_1x04, symbol CONN_4
- added R11: 33k, symbol R
- added R4: 3k3, symbol R
- added SW2: SW_Push, symbol SW_Push
- added unit 4 of U4
- C1: value CP -> 100nF
- C3: renamed from C2; value CP -> 1uF
- C7: renamed from C6; value CP -> 0.33uF
- C8: renamed from C7; value CP -> 1uF
- CON1: footprint AVR-ISP-10 -> Connect:IDC_Header_Straight_10pins
- D1: footprint (none) -> Diodes_ThroughHole:Diode_P600_Vertical_AnodeUp
- J1: footprint (none) -> Connect:BARREL_JACK
- JP1: footprint (none) -> Pin_Headers:Pin_Header_Straight_1x03
- P1: footprint (none) -> Pin_Headers:Pin_Header_Straight_1x04
- P2: footprint (none) -> Connect:AK300-2
- R1, R2, R3: footprint Resistors_SMD:R_0805 -> (none)
- R10: renamed from R9; footprint Resistors_SMD:R_0805 -> (none)
- R12: renamed from R10; footprint Resistors_SMD:R_0805 -> (none)
- R13: renamed from R11; footprint Resistors_SMD:R_0805 -> (none)
- R14: renamed from R12; footprint Resistors_SMD:R_0805 -> (none)
- R5: renamed from R4; footprint Resistors_SMD:R_0805 -> (none)
- R6: renamed from R5; footprint Resistors_SMD:R_0805 -> (none)
- R7: renamed from R6; footprint Resistors_SMD:R_0805 -> (none)
- R8: renamed from R7; footprint Resistors_SMD:R_0805 -> (none)
- R9: renamed from R8; footprint Resistors_SMD:R_0805 -> (none)
- U3: footprint Housings_DIP:DIP-8_W7.62mm -> (none)
- gave numbers to parts that had none: 2
- renumbered C3 to C4, C4 to C5, C5 to C6, C8 to C9
Connections:
- net 5V: now also R11.1
- net GND: now also P3.4 (P4), SW2.2, U4.7 (GND)
- net VCC: now also U4.14 (VCC)
- net Vin: now also J1.1 (P1), R1.2
- net at U3.3 (PB4(ADC2/PCINT4)): now also U4.8
- net at Q5.3 (S), R14.1: now also P3.1 (P1), P3.2 (P2)
- new net: R11.2, R4.2, SW2.1
- new net: C2.1, R4.1, U4.9
- no-connect marks 2 -> 3
Other:
- moved on the sheet: C4, C5, C6, R5, R6, R7, SW1, U4A, U4B, U4C

Commit message: ...
Parts:
- removed R2: 240, symbol R
- removed R3: 750, symbol R
- added C4: 100nF, Capacitors_SMD:C_0805, symbol C
- C1: value 100nF -> 1uF; footprint (none) -> Capacitors_SMD:C_0805
- C10: renamed from C9; footprint (none) -> Capacitors_THT:CP_Radial_D16.0mm_P7.50mm
- C11: renamed from C10; footprint (none) -> Capacitors_SMD:C_0805
- C12: renamed from C11; footprint (none) -> Capacitors_SMD:C_0805
- C2: renamed from C3; footprint (none) -> Capacitors_SMD:C_0805
- C3: renamed from C2; value C -> 10n; footprint (none) -> Capacitors_SMD:C_0805
- C5: renamed from C4; footprint (none) -> Capacitors_SMD:C_0805
- C6: renamed from C5; footprint (none) -> Capacitors_SMD:C_0805
- C7: renamed from C6; footprint (none) -> Capacitors_SMD:C_0805
- C8: renamed from C7; value 0.33uF -> 1uF; footprint (none) -> Capacitors_SMD:C_0805
- C9: renamed from C8; footprint (none) -> Capacitors_SMD:C_0805
- CON1: footprint Connect:IDC_Header_Straight_10pins -> Connectors:IDC_Header_Straight_10pins
- D1: footprint Diodes_ThroughHole:Diode_P600_Vertical_AnodeUp -> Diodes_THT:D_DO-27_P5.08mm_Vertical_AnodeUp
- J1: footprint Connect:BARREL_JACK -> Connectors:BARREL_JACK
- JP1: footprint Pin_Headers:Pin_Header_Straight_1x03 -> Pin_Headers:Pin_Header_Angled_1x03_Pitch2.54mm
- P1: footprint Pin_Headers:Pin_Header_Straight_1x04 -> Pin_Headers:Pin_Header_Angled_1x04_Pitch2.54mm
- P2: footprint Connect:AK300-2 -> Connectors:AK300-2
- P3: footprint Pin_Headers:Pin_Header_Angled_1x04 -> Pin_Headers:Pin_Header_Angled_1x04_Pitch2.54mm
- Q1, Q2, Q3, Q4: footprint (none) -> TO_SOT_Packages_THT:TO-92_Inline_Wide
- Q5: footprint (none) -> myLib:TO-220-3
- R1: footprint (none) -> Resistors_SMD:R_0805
- R10: renamed from R12; footprint (none) -> Resistors_SMD:R_0805
- R11: renamed from R13; footprint (none) -> Resistors_SMD:R_0805
- R12: renamed from R14; footprint (none) -> myLib:SolderWirePad_2x_1-5mmDrill
- R2: renamed from R4; footprint (none) -> Resistors_SMD:R_0805
- R3: renamed from R5; footprint (none) -> Resistors_SMD:R_0805
- R4: renamed from R6; footprint (none) -> Resistors_SMD:R_0805
- R5: renamed from R7; footprint (none) -> Resistors_SMD:R_0805
- R6: renamed from R8; footprint (none) -> Resistors_SMD:R_0805
- R7: renamed from R9; footprint (none) -> Resistors_SMD:R_0805
- R8: renamed from R10; footprint (none) -> Resistors_SMD:R_0805
- R9: renamed from R11; footprint (none) -> Resistors_SMD:R_0805
- SW1: footprint (none) -> myLib:PEC11_Switch_Rotary_Encoder
- SW2: footprint (none) -> Buttons_Switches_THT:SW_PUSH_6mm
- U1: value LM317LZ -> 78L_REG; footprint (none) -> TO_SOT_Packages_THT:TO-92_Inline_Wide
- U2: value 78L15 -> 78L_REG; footprint (none) -> TO_SOT_Packages_THT:TO-92_Inline_Wide
- U3: footprint (none) -> Housings_DIP:DIP-8_W7.62mm
- U4: footprint (none) -> Housings_DIP:DIP-14_W7.62mm_Socket
Connections:
- net 15V: now also Q4.3 (C)
- net GND: now also C3.2, CON1.10, Q3.3 (C), U1.2 (GND), C4.2; no longer Q4.1 (E)
- net at Q3.1 (E), Q5.1 (G): now also Q4.1 (E); no longer Q4.3 (C)
- net 5V renamed +5V
- net +5V: now also C4.1
Other:
- moved on the sheet: C2, Q3, Q4, R1
